File: pcb/RoyTyper.kicad_pcb (KiCad board)
At the start: 2 copper layers, 99.2 x 63.9 mm, 23 parts, among them SW1 SW_Push_45deg, SW11 RotaryEncoder_Switch, SW2 SW_Push_45deg, SW3 SW_Push_45deg, SW4 SW_Push_45deg, SW5 SW_Push_45deg, SW6 SW_Push_45deg, SW7 SW_Push_45deg, SW8 SW_Push_45deg, SW9 SW_Push_45deg, U1 XIAO-RP2040-DIP

Commit message: Fixed a minor error, and updated screenshot
Other:
- board size 99.2 x 63.9 mm -> 99.2 x 64 mm
- board text added: "RoyTyper"
- board text removed: "RoyTyper:)"
Changed lines of the file:
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@@
 			)
 		)
-		(model "${KIPRJMOD}/3D/SK6812_Mini.step"
+		(model "${KIPRJMOD}/assets/3D/SK6812_Mini.step"
 			(offset
 				(xyz 0 0 0)
@@
 			)
 		)
-		(model "${KIPRJMOD}/3D/SW_Cherry_MX_PCB.stp"
+		(model "${KIPRJMOD}/assets/3D/SW_Cherry_MX_PCB.stp"
 			(offset
 				(xyz -2.5 -5 0)
@@
 			)
 		)
-		(model "${KIPRJMOD}/3D/SW_Cherry_MX_PCB.stp"
+		(model "${KIPRJMOD}/assets/3D/SW_Cherry_MX_PCB.stp"
 			(offset
 				(xyz -2.5 -5 0)
@@
 			)
 		)
-		(model "${KIPRJMOD}/3D/SW_Cherry_MX_PCB.stp"
+		(model "${KIPRJMOD}/assets/3D/SW_Cherry_MX_PCB.stp"
 			(offset
 				(xyz -2.5 -5 0)
@@
 			)
 		)
-		(model "${KIPRJMOD}/3D/SW_Cherry_MX_PCB.stp"
+		(model "${KIPRJMOD}/assets/3D/SW_Cherry_MX_PCB.stp"
 			(offset
 				(xyz -2.5 -5 0)
@@
 			)
 		)
-		(model "${KIPRJMOD}/3D/SW_Cherry_MX_PCB.stp"
+		(model "${KIPRJMOD}/assets/3D/SW_Cherry_MX_PCB.stp"
 			(offset
 				(xyz -2.5 -5 0)
@@
 			)
 		)
-		(model "${KIPRJMOD}/3D/SW_Cherry_MX_PCB.stp"
+		(model "${KIPRJMOD}/assets/3D/SW_Cherry_MX_PCB.stp"
 			(offset
 				(xyz -2.5 -5 0)
@@
 			)
 		)
-		(model "${KIPRJMOD}/3D/RotaryEncoder_Alps_EC11E-Switch_Vertical_H20mm.step"
+		(model "${KIPRJMOD}/assets/3D/RotaryEncoder_Alps_EC11E-Switch_Vertical_H20mm.step"
 			(offset
 				(xyz 0 0 0)
@@
 			)
 		)
-		(model "${KIPRJMOD}/3D/SW_Cherry_MX_PCB.stp"
+		(model "${KIPRJMOD}/assets/3D/SW_Cherry_MX_PCB.stp"
 			(offset
 				(xyz -2.5 -5 0)
@@
 			)
 		)
-		(model "${KIPRJMOD}/3D/SW_Cherry_MX_PCB.stp"
+		(model "${KIPRJMOD}/assets/3D/SW_Cherry_MX_PCB.stp"
 			(offset
 				(xyz -2.5 -5 0)
@@
 			)
 		)
-		(model "${KIPRJMOD}/3D/SK6812_Mini.step"
+		(model "${KIPRJMOD}/assets/3D/SK6812_Mini.step"
 			(offset
 				(xyz 0 0 0)
@@
 			)
 		)
-		(model "${KIPRJMOD}/3D/SW_Cherry_MX_PCB.stp"
+		(model "${KIPRJMOD}/assets/3D/SW_Cherry_MX_PCB.stp"
 			(offset
 				(xyz -2.5 -5 0)
@@
 			)
 		)
-		(model "${KIPRJMOD}/3D/SK6812_Mini.step"
+		(model "${KIPRJMOD}/assets/3D/SK6812_Mini.step"
 			(offset
 				(xyz 0 0 0)
@@
 		(at 79.845 67.945)
 		(property "Reference" "U1"
-			(at -8.5 -12 0)
+			(at -0.4 -1.83 0)
 			(unlocked yes)
 			(layer "F.SilkS")
 			(effects
 				(font
-					(size 0.635 0.635)
+					(size 0.82 0.635)
 					(thickness 0.1016)
 				)
@@
 		)
 		(model "${AMZPATH}/3dmodels/AMz3D.3dshapes/Seeeduino XIAO SAMD21 v4.step"
+			(hide yes)
 			(offset
 				(xyz 0 0 0)
@@
 			)
 		)
-		(model "${KIPRJMOD}/3D/seed.step"
+		(model "${KIPRJMOD}/assets/3D/seed.step"
 			(offset
 				(xyz 0 0 0)
@@
 			)
 		)
-		(fp_text user "${REFERENCE}"
-			(at 4.11 0 -90)
+		(fp_text user "K"
+			(at 0 1.8 -90)
 			(layer "B.Fab")
 			(effects
 				(font
-					(size 0.8 0.8)
-					(thickness 0.12)
+					(size 1 1)
+					(thickness 0.15)
 				)
 				(justify mirror)
 			)
 		)
-		(fp_text user "K"
-			(at 0 1.8 -90)
+		(fp_text user "${REFERENCE}"
+			(at 4.11 0 -90)
 			(layer "B.Fab")
 			(effects
 				(font
-					(size 1 1)
-					(thickness 0.15)
+					(size 0.8 0.8)
+					(thickness 0.12)
 				)
 				(justify mirror)
@@
 			)
 		)
-		(fp_text user "${REFERENCE}"
-			(at 4.11 0 -90)
+		(fp_text user "K"
+			(at 0 1.8 -90)
 			(layer "B.Fab")
 			(effects
 				(font
-					(size 0.8 0.8)
-					(thickness 0.12)
+					(size 1 1)
+					(thickness 0.15)
 				)
 				(justify mirror)
 			)
 		)
-		(fp_text user "K"
-			(at 0 1.8 -90)
+		(fp_text user "${REFERENCE}"
+			(at 4.11 0 -90)
 			(layer "B.Fab")
 			(effects
 				(font
-					(size 1 1)
-					(thickness 0.15)
+					(size 0.8 0.8)
+					(thickness 0.12)
 				)
 				(justify mirror)
@@
 			)
 		)
-		(fp_text user "K"
-			(at 0 1.8 -90)
+		(fp_text user "${REFERENCE}"
+			(at 4.11 0 -90)
 			(layer "B.Fab")
 			(effects
 				(font
-					(size 1 1)
-					(thickness 0.15)
+					(size 0.8 0.8)
+					(thickness 0.12)
 				)
 				(justify mirror)
 			)
 		)
-		(fp_text user "${REFERENCE}"
-			(at 4.11 0 -90)
+		(fp_text user "K"
+			(at 0 1.8 -90)
 			(layer "B.Fab")
 			(effects
 				(font
-					(size 0.8 0.8)
-					(thickness 0.12)
+					(size 1 1)
+					(thickness 0.15)
 				)
 				(justify mirror)
@@
 	)
 	(gr_rect
-		(start 53.215 57.345)
+		(start 53.215 57.265)
 		(end 152.445 121.285)
 		(stroke
@@
 		(layer "Edge.Cuts")
 	)
-	(gr_text "RoyTyper:)"
-		(at 80.105 61.525 -0)
-		(layer "Edge.Cuts")
+	(gr_text "RoyTyper"
+		(at 76.485 62.085 0)
+		(layer "F.SilkS")
 		(effects
 			(font
 				(size 1 1)
-				(thickness 0.15)
+				(thickness 0.1)
 			)
 			(justify left bottom)
